Commit message: fixes

File: test_car.urdf (robot description, URDF)
Before this commit: robot fsd_car, 7 links, 6 joints
Links:
- link base_link: geometry collision box size=1.0 0.5 0.2; visual box size=1.0 0.5 0.2
- link left_wheel: geometry collision cylinder length=0.1 radius=0.15; visual cylinder length=0.1 radius=0.15
- link right_wheel: geometry collision cylinder length=0.1 radius=0.15; visual cylinder length=0.1 radius=0.15
Joints:
- joint base_footprint_joint: origin xyz=0 0 ${wheel_radius + base_height/2} rpy=0 0 0 -> xyz=0 0 0.25 rpy=0 0 0
- joint camera_left_joint: origin xyz=${base_length/2 - 0.05} 0.06 0.50 rpy=0 ${-15*pi/180} 0 -> xyz=0.45 0.06 0.50 rpy=0 -0.26179916666666664 0
- joint caster_wheel_joint: origin xyz=0.3 0 ${-base_height/2 - 0.05} rpy=0 0 0 -> xyz=0.3 0 -0.15000000000000002 rpy=0 0 0
- joint laser_joint: origin xyz=${base_length/2 - 0.1} 0 0.15 rpy=0 0 0 -> xyz=0.4 0 0.15 rpy=0 0 0
- joint left_wheel_joint: origin xyz=-0.2 ${base_width/2 + wheel_width/2} ${-base_height/2} rpy=${-pi/2} 0 0 -> xyz=-0.2 0.3 -0.1 rpy=-1.570795 0 0
- joint right_wheel_joint: origin xyz=-0.2 ${-base_width/2 - wheel_width/2} ${-base_height/2} rpy=${-pi/2} 0 0 -> xyz=-0.2 -0.3 -0.1 rpy=-1.570795 0 0
