Commit message: fixes in lidar and stereo camera

File: src/fsd_perception/urdf/fsd_car.urdf.xacro (robot description, xacro)
@@ -118,89 +118,45 @@
     <origin xyz="${base_length/2 - 0.05} 0.06 0.50" rpy="0 ${-15*pi/180} 0"/>
   </joint>
-  <gazebo reference="camera_left_link">
-    <sensor type="camera" name="camera_left">
-      <update_rate>30.0</update_rate>
-      <camera name="left">
-        <horizontal_fov>1.91986</horizontal_fov>
-        <image>
-          <width>1280</width>
-          <height>720</height>
-          <format>R8G8B8</format>
-        </image>
-        <clip>
-          <near>0.1</near>
-          <far>100</far>
-        </clip>
-        <noise>
-          <type>gaussian</type>
-          <mean>0.0</mean>
-          <stddev>0.007</stddev>
-        </noise>
-      </camera>
-      <plugin name="camera_left_controller" filename="libgazebo_ros_camera.so">
-        <alwaysOn>true</alwaysOn>
-        <updateRate>30.0</updateRate>
-        <cameraName>camera_left</cameraName>
-        <imageTopicName>/camera/left/image_raw</imageTopicName>
-        <cameraInfoTopicName>/camera/left/camera_info</cameraInfoTopicName>
-        <frameName>camera_left_link</frameName>
-      </plugin>
-    </sensor>
-  </gazebo>
-  <!-- Right camera -->
-  <link name="camera_right_link">
-    <visual>
-      <geometry>
-        <box size="0.03 0.03 0.03"/>
-      </geometry>
-      <material name="red">
-        <color rgba="1 0 0 1"/>
-      </material>
-    </visual>
-    <collision>
-      <geometry>
-        <box size="0.03 0.03 0.03"/>
-      </geometry>
-    </collision>
-    <inertial>
-      <mass value="0.05"/>
-      <inertia ixx="0.0001" ixy="0.0" ixz="0.0" iyy="0.0001" iyz="0.0" izz="0.0001"/>
-    </inertial>
-  </link>
-  <joint name="camera_right_joint" type="fixed">
-    <parent link="base_link"/>
-    <child link="camera_right_link"/>
-    <origin xyz="${base_length/2 - 0.05} -0.06 0.50" rpy="0 ${-15*pi/180} 0"/>
-  </joint>
-  <gazebo reference="camera_right_link">
-    <sensor type="camera" name="camera_right">
-      <update_rate>30.0</update_rate>
-      <camera name="right">
-        <horizontal_fov>1.91986</horizontal_fov>
-        <image>
-          <width>1280</width>
-          <height>720</height>
-          <format>R8G8B8</format>
-        </image>
-        <clip>
-          <near>0.1</near>
-          <far>100</far>
-        </clip>
-        <noise>
-          <type>gaussian</type>
-          <mean>0.0</mean>
-          <stddev>0.007</stddev>
-        </noise>
-      </camera>
-      <plugin name="camera_right_controller" filename="libgazebo_ros_camera.so">
-        <alwaysOn>true</alwaysOn>
-        <updateRate>30.0</updateRate>
-        <cameraName>camera_right</cameraName>
-        <imageTopicName>/camera/right/image_raw</imageTopicName>
-        <cameraInfoTopicName>/camera/right/camera_info</cameraInfoTopicName>
-        <frameName>camera_right_link</frameName>
-      </plugin>
-    </sensor>
-  </gazebo>
+<gazebo reference="camera_left_link">
+  <sensor type="multicamera" name="zed_stereo_sensor">
+    <update_rate>30.0</update_rate>
+    <camera name="left">
+      <horizontal_fov>1.91986</horizontal_fov>
+      <image>
+        <width>1280</width>
+        <height>720</height>
+        <format>R8G8B8</format>
+      </image>
+      <clip><near>0.1</near><far>100</far></clip>
+    </camera>
+    <camera name="right">
+      <horizontal_fov>1.91986</horizontal_fov>
+      <image>
+        <width>1280</width>
+        <height>720</height>
+        <format>R8G8B8</format>
+      </image>
+      <clip><near>0.1</near><far>100</far></clip>
+      <pose>0 -0.12 0 0 0 0</pose>
+    </camera>
+    <plugin name="stereo_camera_controller" filename="libgazebo_ros_multicamera.so">
+      <alwaysOn>true</alwaysOn>
+      <updateRate>30.0</updateRate>
+      <cameraName>zed</cameraName>
+      <imageTopicName>rgb/image_raw</imageTopicName>
+      <cameraInfoTopicName>rgb/camera_info</cameraInfoTopicName>
+      <frameName>camera_left_link</frameName>
+      <hackBaseline>0.12</hackBaseline> </plugin>
+    <plugin name="stereo_point_cloud_controller" filename="libgazebo_ros_openni_kinect.so">
+      <alwaysOn>true</alwaysOn>
+      <updateRate>30.0</updateRate>
+      <cameraName>zed</cameraName>
+      <imageTopicName>depth/image_raw</imageTopicName>
+      <cameraInfoTopicName>depth/camera_info</cameraInfoTopicName>
+      <pointCloudTopic>point_cloud/cloud_registered</pointCloudTopic> <frameName>camera_left_link</frameName>
+      <depthImage>true</depthImage>
+    </plugin>
+  </sensor>
+</gazebo>
   <!-- Gazebo appearance -->
   <gazebo reference="base_link">

Commit message: car fixes

File: src/fsd_perception/urdf/fsd_car.urdf.xacro (robot description, xacro)
@@ -1,5 +1,4 @@
 <?xml version="1.0"?>
 <robot name="fsd_car" xmlns:xacro="http://www.ros.org/wiki/xacro">
-  <!-- Properties -->
   <xacro:property name="base_width" value="0.5"/>
   <xacro:property name="base_length" value="1.0"/>
@@ -8,5 +7,4 @@
   <xacro:property name="wheel_width" value="0.1"/>
   <xacro:property name="pi" value="3.14159"/>
-  <!-- Base Link -->
   <link name="base_link">
     <visual>
@@ -28,5 +26,4 @@
     </inertial>
   </link>
-  <!-- Footprint -->
   <link name="base_footprint"/>
   <joint name="base_footprint_joint" type="fixed">
@@ -35,5 +32,4 @@
     <origin xyz="0 0 ${wheel_radius + base_height/2}" rpy="0 0 0"/>
   </joint>
-  <!-- ========== 2D LIDAR ========== -->
   <link name="laser_link">
     <visual>
@@ -60,5 +56,4 @@
     <origin xyz="${base_length/2 - 0.1} 0 0.15" rpy="0 0 0"/>
   </joint>
-  <!-- LiDAR Sensor Plugin -->
   <gazebo reference="laser_link">
     <sensor type="ray" name="lidar_sensor">
@@ -92,6 +87,4 @@
     </sensor>
   </gazebo>
-  <!-- ========== STEREO CAMERAS ========== -->
-  <!-- Left camera -->
   <link name="camera_left_link">
     <visual>
@@ -150,119 +143,3 @@
   </sensor>
 </gazebo>
-  <!-- Gazebo appearance -->
-  <gazebo reference="base_link">
-    <material>Gazebo/Blue</material>
-  </gazebo>
-  <!-- Differential Drive Plugin -->
-  <gazebo>
-    <plugin name="differential_drive_controller" filename="libgazebo_ros_diff_drive.so">
-      <updateRate>50</updateRate>
-      <leftJoint>left_wheel_joint</leftJoint>
-      <rightJoint>right_wheel_joint</rightJoint>
-      <wheelSeparation>${base_width + wheel_width}</wheelSeparation>
-      <wheelDiameter>${wheel_radius * 2}</wheelDiameter>
-      <wheelAcceleration>1.0</wheelAcceleration>
-      <wheelTorque>20</wheelTorque>
-      <commandTopic>cmd_vel</commandTopic>
-      <odometryTopic>odom</odometryTopic>
-      <odometryFrame>odom</odometryFrame>
-      <robotBaseFrame>base_footprint</robotBaseFrame>
-      <publishWheelTF>true</publishWheelTF>
-      <publishOdomTF>true</publishOdomTF>
-      <publishWheelJointState>true</publishWheelJointState>
-      <legacyMode>false</legacyMode>
-      <rosDebugLevel>na</rosDebugLevel>
-    </plugin>
-  </gazebo>
-  <!-- Left wheel -->
-  <link name="left_wheel">
-    <visual>
-      <geometry>
-        <cylinder radius="${wheel_radius}" length="${wheel_width}"/>
-      </geometry>
-      <material name="black"/>
-    </visual>
-    <collision>
-      <geometry>
-        <cylinder radius="${wheel_radius}" length="${wheel_width}"/>
-      </geometry>
-    </collision>
-    <inertial>
-      <mass value="1"/>
-      <inertia ixx="0.01" ixy="0.0" ixz="0.0" iyy="0.01" iyz="0.0" izz="0.01"/>
-    </inertial>
-  </link>
-  <joint name="left_wheel_joint" type="continuous">
-    <parent link="base_link"/>
-    <child link="left_wheel"/>
-    <origin xyz="-0.2 ${base_width/2 + wheel_width/2} ${-base_height/2}" rpy="${-pi/2} 0 0"/>
-    <axis xyz="0 0 1"/>
-  </joint>
-  <!-- Right wheel -->
-  <link name="right_wheel">
-    <visual>
-      <geometry>
-        <cylinder radius="${wheel_radius}" length="${wheel_width}"/>
-      </geometry>
-      <material name="black"/>
-    </visual>
-    <collision>
-      <geometry>
-        <cylinder radius="${wheel_radius}" length="${wheel_width}"/>
-      </geometry>
-    </collision>
-    <inertial>
-      <mass value="1"/>
-      <inertia ixx="0.01" ixy="0.0" ixz="0.0" iyy="0.01" iyz="0.0" izz="0.01"/>
-    </inertial>
-  </link>
-  <joint name="right_wheel_joint" type="continuous">
-    <parent link="base_link"/>
-    <child link="right_wheel"/>
-    <origin xyz="-0.2 ${-base_width/2 - wheel_width/2} ${-base_height/2}" rpy="${-pi/2} 0 0"/>
-    <axis xyz="0 0 1"/>
-  </joint>
-  <!-- Caster wheel -->
-  <link name="caster_wheel">
-    <visual>
-      <geometry>
-        <sphere radius="0.05"/>
-      </geometry>
-      <material name="black"/>
-    </visual>
-    <collision>
-      <geometry>
-        <sphere radius="0.05"/>
-      </geometry>
-    </collision>
-    <inertial>
-      <mass value="0.5"/>
-      <inertia ixx="0.001" ixy="0.0" ixz="0.0" iyy="0.001" iyz="0.0" izz="0.001"/>
-    </inertial>
-  </link>
-  <joint name="caster_wheel_joint" type="fixed">
-    <parent link="base_link"/>
-    <child link="caster_wheel"/>
-    <origin xyz="0.3 0 ${-base_height/2 - 0.05}" rpy="0 0 0"/>
-  </joint>
-  <!-- Gazebo properties -->
-  <gazebo reference="left_wheel">
-    <material>Gazebo/Black</material>
-    <mu1>1.0</mu1>
-    <mu2>1.0</mu2>
-    <kp>1000000.0</kp>
-    <kd>100.0</kd>
-  </gazebo>
-  <gazebo reference="right_wheel">
-    <material>Gazebo/Black</material>
-    <mu1>1.0</mu1>
-    <mu2>1.0</mu2>
-    <kp>1000000.0</kp>
-    <kd>100.0</kd>
-  </gazebo>
-  <gazebo reference="caster_wheel">
-    <material>Gazebo/Black</material>
-    <mu1>0.0</mu1>
-    <mu2>0.0</mu2>
-  </gazebo>
 </robot>
